File: custom_board.kicad_pcb (KiCad board)
At the start: 2 copper layers, 4 parts, among them IC1 TMPM46BF10FG

Commit message: idk
Parts:
- added C10: .1u, Capacitor_SMD:C_0805_2012Metric, F.Cu at (188.2, 110.9)
- added C11: .1u, Capacitor_SMD:C_0805_2012Metric, B.Cu at (152.2, 97.3)
- added C12: .1u, Capacitor_SMD:C_0805_2012Metric, F.Cu at (187.2, 106.3)
- added C13: 10p, Capacitor_SMD:C_0805_2012Metric, F.Cu at (139.6, 138.1)
- added C14: 10p, Capacitor_SMD:C_0805_2012Metric, F.Cu at (234.4, 102.5)
- added C15: .1u, Capacitor_SMD:C_0805_2012Metric, F.Cu at (202.1, 123.8)
- added C4: 10p, Capacitor_SMD:C_0805_2012Metric, B.Cu at (144.8, 84.0)
- added C5: 10p, Capacitor_SMD:C_0805_2012Metric, F.Cu at (181.8, 111.4)
- added C6: .1u, Capacitor_SMD:C_0805_2012Metric, B.Cu at (152.2, 100.7)
- added C7: .1u, Capacitor_SMD:C_0805_2012Metric, F.Cu at (184.5, 102.7)
- added C8: .1u, Capacitor_SMD:C_0805_2012Metric, F.Cu at (242.7, 119.2)
- added C9: .1u, Capacitor_SMD:C_0805_2012Metric, B.Cu at (144.8, 98.9)
- added J1: USB_UART Conn Pins, Connector_PinSocket_2.54mm:PinSocket_1x05_P2.54mm_Horizontal, F.Cu at (94.1, 93.5)
- added J10: Port C, Connector_PinSocket_2.54mm:PinSocket_1x06_P2.54mm_Vertical, F.Cu at (213.3, 63.3)
- added J11: Port F, Connector_PinSocket_2.54mm:PinSocket_1x08_P2.54mm_Vertical, F.Cu at (194.9, 63.3)
- added J12: Port J, Connector_PinSocket_2.54mm:PinSocket_1x08_P2.54mm_Vertical, F.Cu at (185.7, 63.3)
- added J2: Port G, Connector_PinSocket_2.54mm:PinSocket_1x08_P2.54mm_Vertical, F.Cu at (204.1, 63.3)
- added J3: Port A, Connector_PinSocket_2.54mm:PinSocket_1x08_P2.54mm_Vertical, F.Cu at (199.5, 63.3)
- added J4: Port D, Connector_PinSocket_2.54mm:PinSocket_1x05_P2.54mm_Vertical, F.Cu at (222.5, 63.3)
- added J5: Port K, Connector_PinSocket_2.54mm:PinSocket_1x05_P2.54mm_Vertical, F.Cu at (217.9, 63.3)
- added J6: Port L, Connector_PinSocket_2.54mm:PinSocket_1x04_P2.54mm_Vertical, F.Cu at (216.6, 84.5)
- added J7: Port E, Connector_PinSocket_2.54mm:PinSocket_1x08_P2.54mm_Vertical, F.Cu at (190.3, 63.3)
- added J8: Port H, Connector_PinSocket_2.54mm:PinSocket_1x04_P2.54mm_Vertical, F.Cu at (241.0, 63.3)
- added J9: Port B, Connector_PinSocket_2.54mm:PinSocket_1x08_P2.54mm_Vertical, F.Cu at (208.7, 63.3)
- added R1: 47, Resistor_SMD:R_0805_2012Metric_Pad1.20x1.40mm_HandSolder, F.Cu at (216.7, 95.9)
- added R2: 10k, Resistor_SMD:R_0805_2012Metric_Pad1.20x1.40mm_HandSolder, F.Cu at (221.3, 83.7)
- added R3: 10k, Resistor_SMD:R_0805_2012Metric_Pad1.20x1.40mm_HandSolder, F.Cu at (218.2, 110.2)
- added SW1: Boot Switch, Button_Switch_SMD:SW_DIP_SPSTx01_Slide_9.78x4.72mm_W8.61mm_P2.54mm, F.Cu at (89.4, 114.6)
- added SW2: SW_Push, Button_Switch_THT:Push_E-Switch_KS01Q01, F.Cu at (86.6, 125.7)
- added Y1: HighOscillator, Crystal:Crystal_SMD_Abracon_ABM10-4Pin_2.5x2.0mm, F.Cu at (225.7, 84.5)
- added Y2: LowOscillator, Crystal:Crystal_SMD_EuroQuartz_EQ161-2Pin_3.2x1.5mm_HandSoldering, F.Cu at (231.6, 76.0)
- C2: moved to B.Cu
- moved C3 73.1 mm to (139.6, 135.1)
- moved C1 67.9 mm to (144.1, 135.1)
- moved C2 50.6 mm to (148.6, 105.4)
- moved IC1 8.89 mm to (147.3, 95.0)
Connections:
- IC1 pad 1: unconnected-(IC1-Pad1) -> PJ0
- IC1 pad 100: GNDA -> RVSS
- IC1 pad 13: unconnected-(IC1-Pad13) -> PE0
- IC1 pad 14: unconnected-(IC1-Pad14) -> PE1_RXD0
- IC1 pad 15: unconnected-(IC1-Pad15) -> PE2_TXD0
- IC1 pad 16: unconnected-(IC1-Pad16) -> PE3
- IC1 pad 17: unconnected-(IC1-Pad17) -> PE4
- IC1 pad 18: unconnected-(IC1-Pad18) -> PE5
- IC1 pad 19: unconnected-(IC1-Pad19) -> PE6
- IC1 pad 2: unconnected-(IC1-Pad2) -> PJ1
- IC1 pad 20: unconnected-(IC1-Pad20) -> PE7
- IC1 pad 23: unconnected-(IC1-Pad23) -> PF0
- IC1 pad 24: unconnected-(IC1-Pad24) -> PF1
- IC1 pad 25: unconnected-(IC1-Pad25) -> PF2
- IC1 pad 26: unconnected-(IC1-Pad26) -> PF3
- IC1 pad 27: unconnected-(IC1-Pad27) -> PF4
- IC1 pad 28: unconnected-(IC1-Pad28) -> PF5
- IC1 pad 29: unconnected-(IC1-Pad29) -> PF6
- IC1 pad 3: unconnected-(IC1-Pad3) -> PJ2
- IC1 pad 30: unconnected-(IC1-Pad30) -> PF7
- IC1 pad 31: unconnected-(IC1-Pad31) -> PG0
- IC1 pad 32: unconnected-(IC1-Pad32) -> PG1
- IC1 pad 33: unconnected-(IC1-Pad33) -> PG2
- IC1 pad 34: unconnected-(IC1-Pad34) -> PG3
- IC1 pad 35: unconnected-(IC1-Pad35) -> PG4
- IC1 pad 36: unconnected-(IC1-Pad36) -> PG5
- IC1 pad 37: unconnected-(IC1-Pad37) -> PG6
- IC1 pad 38: unconnected-(IC1-Pad38) -> PG7
- IC1 pad 4: unconnected-(IC1-Pad4) -> PJ3
- IC1 pad 43: unconnected-(IC1-Pad43) -> PB2
- IC1 pad 44: unconnected-(IC1-Pad44) -> PB3
- IC1 pad 45: unconnected-(IC1-Pad45) -> PB4
- IC1 pad 46: unconnected-(IC1-Pad46) -> PB5
- IC1 pad 47: unconnected-(IC1-Pad47) -> Net-(IC1-Pad47)
- IC1 pad 48: unconnected-(IC1-Pad48) -> PB7
- IC1 pad 49: unconnected-(IC1-Pad49) -> PB8
- IC1 pad 5: unconnected-(IC1-Pad5) -> PJ4
- IC1 pad 50: unconnected-(IC1-Pad50) -> PB9
- IC1 pad 51: unconnected-(IC1-Pad51) -> PH1
- IC1 pad 52: unconnected-(IC1-Pad52) -> PH0
- IC1 pad 53: unconnected-(IC1-Pad53) -> PD4
- IC1 pad 54: unconnected-(IC1-Pad54) -> PD3
- IC1 pad 55: unconnected-(IC1-Pad55) -> PD2
- IC1 pad 56: unconnected-(IC1-Pad56) -> PD1
- IC1 pad 57: unconnected-(IC1-Pad57) -> PD0
- IC1 pad 58: unconnected-(IC1-Pad58) -> Net-(IC1-Pad58)
- IC1 pad 59: unconnected-(IC1-Pad59) -> Net-(C13-Pad1)
- IC1 pad 6: unconnected-(IC1-Pad6) -> PJ5
- IC1 pad 61: unconnected-(IC1-Pad61) -> Net-(IC1-Pad61)
- IC1 pad 62: unconnected-(IC1-Pad62) -> RVSS
- IC1 pad 65: +3V3 -> RVSS
- IC1 pad 69: unconnected-(IC1-Pad69) -> Net-(C5-Pad1)
- IC1 pad 7: unconnected-(IC1-Pad7) -> PJ6
- IC1 pad 70: unconnected-(IC1-Pad70) -> Net-(C4-Pad1)
- IC1 pad 72: unconnected-(IC1-Pad72) -> PC5
- IC1 pad 73: unconnected-(IC1-Pad73) -> PC4
- IC1 pad 74: unconnected-(IC1-Pad74) -> PC3
- IC1 pad 75: unconnected-(IC1-Pad75) -> PC2
- IC1 pad 76: unconnected-(IC1-Pad76) -> PC1
- IC1 pad 77: unconnected-(IC1-Pad77) -> PC0
- IC1 pad 78: unconnected-(IC1-Pad78) -> PK4
- IC1 pad 79: unconnected-(IC1-Pad79) -> PK3
- IC1 pad 8: unconnected-(IC1-Pad8) -> PJ7
- IC1 pad 80: unconnected-(IC1-Pad80) -> PK2
- IC1 pad 81: unconnected-(IC1-Pad81) -> PK1
- IC1 pad 82: unconnected-(IC1-Pad82) -> PK0
- IC1 pad 83: unconnected-(IC1-Pad83) -> PL0
- IC1 pad 84: unconnected-(IC1-Pad84) -> PL1
- IC1 pad 85: unconnected-(IC1-Pad85) -> PL2
- IC1 pad 86: unconnected-(IC1-Pad86) -> PL3
- IC1 pad 87: unconnected-(IC1-Pad87) -> PB1
- IC1 pad 88: unconnected-(IC1-Pad88) -> PB0
- IC1 pad 91: unconnected-(IC1-Pad91) -> PA7
- IC1 pad 92: unconnected-(IC1-Pad92) -> PA6
- IC1 pad 93: unconnected-(IC1-Pad93) -> PA5
- IC1 pad 94: unconnected-(IC1-Pad94) -> PA4
- IC1 pad 95: unconnected-(IC1-Pad95) -> PA4
- IC1 pad 96: unconnected-(IC1-Pad96) -> PA2
- IC1 pad 97: unconnected-(IC1-Pad97) -> PA1
- IC1 pad 98: unconnected-(IC1-Pad98) -> PA0
Routing:
- net RVSS: track 0.00 -> 97.0 mm, vias 0 -> 9
- net +3V3: track 0.00 -> 7.10 mm, vias 0 -> 1
- net REGIN2: track 0.00 -> 4.62 mm, vias 0 -> 1
- net Net-(C4-Pad1): track 0.00 -> 3.50 mm, vias 0 -> 1
