File: custom_board.kicad_sch (KiCad schematic)
At the start: 34 parts, among them IC1 TMPM46BF10FG, SW1 Boot Switch, SW2 Reset Button, Y1 HighOscillator, Y2 LowOscillator

Commit message: Update custom_board.kicad_sch
Parts:
- gave numbers to parts that had none: 12
Connections:
- net PD0: now also J4.1 (Pin_1)
- net PD1: now also J4.2 (Pin_2)
- net PD2: now also J4.3 (Pin_3)
- net PD3: now also J4.4 (Pin_4)
- net PD4: now also J4.5 (Pin_5)
- net PE0: now also J7.1 (Pin_1)
- net PE3: now also J7.4 (Pin_4)
- net PE4: now also J7.5 (Pin_5)
- net PE5: now also J7.6 (Pin_6)
- net PE6: now also J7.7 (Pin_7)
- net PE7: now also J7.8 (Pin_8)
- net PF0: now also J11.1 (Pin_1)
- net PF1: now also J11.2 (Pin_2)
- net PF2: now also J11.3 (Pin_3)
- net PF3: now also J11.4 (Pin_4)
- net PF4: now also J11.5 (Pin_5)
- net PF5: now also J11.6 (Pin_6)
- net PF6: now also J11.7 (Pin_7)
- net PF7: now also J11.8 (Pin_8)
- net PG0: now also J2.1 (Pin_1)
- net PG1: now also J2.2 (Pin_2)
- net PG2: now also J2.3 (Pin_3)
- net PG3: now also J2.4 (Pin_4)
- net PG4: now also J2.5 (Pin_5)
- net PG5: now also J2.6 (Pin_6)
- net PG6: now also J2.7 (Pin_7)
- net PG7: now also J2.8 (Pin_8)
- net PH0: now also J8.1 (Pin_1)
- net PH1: now also J8.2 (Pin_2)
- net PJ0: now also J12.1 (Pin_1)
- net PJ1: now also J12.2 (Pin_2)
- net PJ2: now also J12.3 (Pin_3)
- net PJ3: now also J12.4 (Pin_4)
- net PJ4: now also J12.5 (Pin_5)
- net PJ5: now also J12.6 (Pin_6)
- net PJ6: now also J12.7 (Pin_7)
- net PJ7: now also J12.8 (Pin_8)
- net PK0: now also J5.1 (Pin_1)
- net PK1: now also J5.2 (Pin_2)
- net PK2: now also J5.3 (Pin_3)
- net PK3: now also J5.4 (Pin_4)
- net PK4: now also J5.5 (Pin_5)
- net PL0: now also J6.1 (Pin_1)
- net PL1: now also J6.2 (Pin_2)
- net PL2: now also J6.3 (Pin_3)
- net PL3: now also J6.4 (Pin_4)
- net RXD0: no longer IC1.14 (PE1)
- net TXD0: no longer IC1.15 (PE2)
- net PE1_RXD0: now reaches J7.2 (Pin_2)
- net PE1_RXD0: now also IC1.14 (PE1)
- net PE2_TXD0: now reaches J7.3 (Pin_3)
- net PE2_TXD0: now also IC1.15 (PE2)
- net PH2: now reaches J8.3 (Pin_3)
- net PH3: now reaches J8.4 (Pin_4)
Other:
- note added: "Datasheet: https://www.mouser.com/datasheet/2/408/TMPM46BF10FG_datasheet_en_20190329-1282396.pdf"
- note added: "Eval board schematic: https://www.sensyst.co.jp/shop/user_data/TMPM46B/TMPM46BF10FG_cir_MP_2.pdf"
- note added: "Parts list on Mouser"
- note added: "Pin Connectors"
- note removed: "https://www.sensyst.co.jp/shop/user_data/TMPM46B/TMPM46BF10FG_cir_MP_2.pdf"

Commit message: Update custom_board.kicad_sch
Parts:
- C10, C11, C12, C13, C14, C4, C5, C6, C7, C8, C9: footprint (none) -> Capacitor_SMD:C_0805_2012Metric
- J1: footprint (none) -> Connector_PinSocket_2.54mm:PinSocket_1x05_P2.54mm_Horizontal
- J10: footprint (none) -> Connector_PinSocket_2.54mm:PinSocket_1x06_P2.54mm_Vertical
- J11, J12, J2, J3, J7, J9: footprint (none) -> Connector_PinSocket_2.54mm:PinSocket_1x08_P2.54mm_Vertical
- J4, J5: footprint (none) -> Connector_PinSocket_2.54mm:PinSocket_1x05_P2.54mm_Vertical
- J6, J8: footprint (none) -> Connector_PinSocket_2.54mm:PinSocket_1x04_P2.54mm_Vertical
- R1, R2, R3: footprint (none) -> Resistor_SMD:R_0805_2012Metric_Pad1.20x1.40mm_HandSolder
- Y1: value HighOscillator -> (none)
- Y2: footprint (none) -> Crystal:Crystal_SMD_EuroQuartz_EQ161-2Pin_3.2x1.5mm_HandSoldering
Changed lines of the file:
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@@
     (property "Reference" "J5" (id 0) (at 311.15 81.28 90))
     (property "Value" "Port K" (id 1) (at 311.15 83.82 90))
-    (property "Footprint" "" (id 2) (at 311.15 86.36 0)
+    (property "Footprint" "Connector_PinSocket_2.54mm:PinSocket_1x05_P2.54mm_Vertical" (id 2) (at 311.15 86.36 0)
       (effects (font (size 1.27 1.27)) hide)
     )
@@
       (effects (font (size 1.27 1.27)) (justify left))
     )
-    (property "Footprint" "" (id 2) (at 202.692 138.43 90)
+    (property "Footprint" "Resistor_SMD:R_0805_2012Metric_Pad1.20x1.40mm_HandSolder" (id 2) (at 202.692 138.43 90)
       (effects (font (size 1.27 1.27)) hide)
     )
@@
       (effects (font (size 1.27 1.27)) (justify left))
     )
-    (property "Footprint" "" (id 2) (at 57.15 26.67 0)
+    (property "Footprint" "Capacitor_SMD:C_0805_2012Metric" (id 2) (at 57.15 26.67 0)
       (effects (font (size 1.27 1.27)) hide)
     )
@@
       (effects (font (size 1.27 1.27)) (justify left))
     )
-    (property "Footprint" "" (id 2) (at 25.4 26.67 0)
+    (property "Footprint" "Capacitor_SMD:C_0805_2012Metric" (id 2) (at 25.4 26.67 0)
       (effects (font (size 1.27 1.27)) hide)
     )
@@
       (effects (font (size 1.27 1.27)) (justify left))
     )
-    (property "Footprint" "" (id 2) (at 15.24 26.67 0)
+    (property "Footprint" "Capacitor_SMD:C_0805_2012Metric" (id 2) (at 15.24 26.67 0)
       (effects (font (size 1.27 1.27)) hide)
     )
@@
     (property "Reference" "C14" (id 0) (at 205.7463 99.06 90))
     (property "Value" "10p" (id 1) (at 205.7463 101.6 90))
-    (property "Footprint" "" (id 2) (at 205.74 105.41 0)
+    (property "Footprint" "Capacitor_SMD:C_0805_2012Metric" (id 2) (at 205.74 105.41 0)
       (effects (font (size 1.27 1.27)) hide)
     )
@@
     (property "Reference" "J7" (id 0) (at 337.82 43.18 90))
     (property "Value" "Port E" (id 1) (at 337.82 45.72 90))
-    (property "Footprint" "" (id 2) (at 336.55 48.26 0)
+    (property "Footprint" "Connector_PinSocket_2.54mm:PinSocket_1x08_P2.54mm_Vertical" (id 2) (at 336.55 48.26 0)
       (effects (font (size 1.27 1.27)) hide)
     )
@@
     (property "Reference" "J11" (id 0) (at 369.57 43.18 90))
     (property "Value" "Port F" (id 1) (at 369.57 45.72 90))
-    (property "Footprint" "" (id 2) (at 368.3 48.26 0)
+    (property "Footprint" "Connector_PinSocket_2.54mm:PinSocket_1x08_P2.54mm_Vertical" (id 2) (at 368.3 48.26 0)
       (effects (font (size 1.27 1.27)) hide)
     )
@@
       (effects (font (size 1.27 1.27)) (justify left))
     )
-    (property "Footprint" "" (id 2) (at 35.56 26.67 0)
+    (property "Footprint" "Capacitor_SMD:C_0805_2012Metric" (id 2) (at 35.56 26.67 0)
       (effects (font (size 1.27 1.27)) hide)
     )
@@
       (effects (font (size 1.27 1.27)) (justify right))
     )
-    (property "Footprint" "" (id 2) (at 200.66 83.82 0)
+    (property "Footprint" "Crystal:Crystal_SMD_EuroQuartz_EQ161-2Pin_3.2x1.5mm_HandSoldering" (id 2) (at 200.66 83.82 0)
       (effects (font (size 1.27 1.27)) hide)
     )
@@
     (property "Reference" "J6" (id 0) (at 336.55 81.28 90))
     (property "Value" "Port L" (id 1) (at 336.55 83.82 90))
-    (property "Footprint" "" (id 2) (at 335.28 86.36 0)
+    (property "Footprint" "Connector_PinSocket_2.54mm:PinSocket_1x04_P2.54mm_Vertical" (id 2) (at 335.28 86.36 0)
       (effects (font (size 1.27 1.27)) hide)
     )
@@
     (property "Reference" "J12" (id 0) (at 369.57 62.23 90))
     (property "Value" "Port J" (id 1) (at 369.57 64.77 90))
-    (property "Footprint" "" (id 2) (at 368.3 67.31 0)
+    (property "Footprint" "Connector_PinSocket_2.54mm:PinSocket_1x08_P2.54mm_Vertical" (id 2) (at 368.3 67.31 0)
       (effects (font (size 1.27 1.27)) hide)
     )
@@
     (property "Reference" "J8" (id 0) (at 339.09 62.23 90))
     (property "Value" "Port H" (id 1) (at 339.09 64.77 90))
-    (property "Footprint" "" (id 2) (at 337.82 67.31 0)
+    (property "Footprint" "Connector_PinSocket_2.54mm:PinSocket_1x04_P2.54mm_Vertical" (id 2) (at 337.82 67.31 0)
       (effects (font (size 1.27 1.27)) hide)
     )
@@
     (property "Reference" "J1" (id 0) (at 24.13 77.47 90))
     (property "Value" "USB_UART Conn Pins" (id 1) (at 24.13 80.01 90))
-    (property "Footprint" "" (id 2) (at 24.13 82.55 0)
+    (property "Footprint" "Connector_PinSocket_2.54mm:PinSocket_1x05_P2.54mm_Horizontal" (id 2) (at 24.13 82.55 0)
       (effects (font (size 1.27 1.27)) hide)
     )
@@
       (effects (font (size 1.27 1.27)) (justify left))
     )
-    (property "Footprint" "" (id 2) (at 160.782 172.72 90)
+    (property "Footprint" "Resistor_SMD:R_0805_2012Metric_Pad1.20x1.40mm_HandSolder" (id 2) (at 160.782 172.72 90)
       (effects (font (size 1.27 1.27)) hide)
     )
@@
       (effects (font (size 1.27 1.27)) (justify left))
     )
-    (property "Footprint" "" (id 2) (at 64.77 26.67 0)
+    (property "Footprint" "Capacitor_SMD:C_0805_2012Metric" (id 2) (at 64.77 26.67 0)
       (effects (font (size 1.27 1.27)) hide)
     )
@@
     (property "Reference" "J3" (id 0) (at 312.42 20.32 90))
     (property "Value" "Port A" (id 1) (at 312.42 22.86 90))
-    (property "Footprint" "" (id 2) (at 311.15 25.4 0)
+    (property "Footprint" "Connector_PinSocket_2.54mm:PinSocket_1x08_P2.54mm_Vertical" (id 2) (at 311.15 25.4 0)
       (effects (font (size 1.27 1.27)) hide)
     )
@@
     (property "Reference" "J2" (id 0) (at 311.15 62.23 90))
     (property "Value" "Port G" (id 1) (at 311.15 64.77 90))
-    (property "Footprint" "" (id 2) (at 309.88 67.31 0)
+    (property "Footprint" "Connector_PinSocket_2.54mm:PinSocket_1x08_P2.54mm_Vertical" (id 2) (at 309.88 67.31 0)
       (effects (font (size 1.27 1.27)) hide)
     )
@@
     (property "Reference" "C4" (id 0) (at 203.2063 74.93 90))
     (property "Value" "10p" (id 1) (at 203.2063 77.47 90))
-    (property "Footprint" "" (id 2) (at 203.2 81.28 0)
+    (property "Footprint" "Capacitor_SMD:C_0805_2012Metric" (id 2) (at 203.2 81.28 0)
       (effects (font (size 1.27 1.27)) hide)
     )
@@
     (property "Reference" "C5" (id 0) (at 203.2 88.9 90))
     (property "Value" "10p" (id 1) (at 203.2 90.17 90))
-    (property "Footprint" "" (id 2) (at 203.2 86.36 0)
+    (property "Footprint" "Capacitor_SMD:C_0805_2012Metric" (id 2) (at 203.2 86.36 0)
       (effects (font (size 1.27 1.27)) hide)
     )
@@
     (property "Reference" "J9" (id 0) (at 342.9 20.32 90))
     (property "Value" "Port B" (id 1) (at 342.9 22.86 90))
-    (property "Footprint" "" (id 2) (at 341.63 25.4 0)
+    (property "Footprint" "Connector_PinSocket_2.54mm:PinSocket_1x08_P2.54mm_Vertical" (id 2) (at 341.63 25.4 0)
       (effects (font (size 1.27 1.27)) hide)
     )
@@
     (property "Reference" "C13" (id 0) (at 203.2 115.57 90))
     (property "Value" "10p" (id 1) (at 203.2 113.03 90))
-    (property "Footprint" "" (id 2) (at 203.2 110.49 0)
+    (property "Footprint" "Capacitor_SMD:C_0805_2012Metric" (id 2) (at 203.2 110.49 0)
       (effects (font (size 1.27 1.27)) hide)
     )
@@
     (property "Reference" "J10" (id 0) (at 369.57 20.32 90))
     (property "Value" "Port C" (id 1) (at 369.57 22.86 90))
-    (property "Footprint" "" (id 2) (at 368.3 25.4 0)
+    (property "Footprint" "Connector_PinSocket_2.54mm:PinSocket_1x06_P2.54mm_Vertical" (id 2) (at 368.3 25.4 0)
       (effects (font (size 1.27 1.27)) hide)
     )
@@
       (effects (font (size 1.27 1.27)) (justify left))
     )
-    (property "Footprint" "" (id 2) (at 45.72 26.67 0)
+    (property "Footprint" "Capacitor_SMD:C_0805_2012Metric" (id 2) (at 45.72 26.67 0)
       (effects (font (size 1.27 1.27)) hide)
     )
@@
     (in_bom yes) (on_board yes)
     (property "Reference" "Y1" (id 0) (at 201.93 104.14 90))
-    (property "Value" "HighOscillator" (id 1) (at 217.17 107.95 90))
+    (property "Value" "" (id 1) (at 217.17 107.95 90))
     (property "Footprint" "" (id 2) (at 199.39 107.95 0)
       (effects (font (size 1.27 1.27)) hide)
     )
-    (property "Datasheet" "https://www.mouser.com/datasheet/2/40/cx2016sa_e-2936404.pdf" (id 3) (at 199.39 107.95 0)
+    (property "Datasheet" "https://www.mouser.com/datasheet/2/3/ABM10AIG-1774860.pdf" (id 3) (at 199.39 107.95 0)
       (effects (font (size 1.27 1.27)) hide)
     )
@@
     (property "Reference" "R1" (id 0) (at 195.58 100.33 90))
     (property "Value" "47" (id 1) (at 195.58 102.87 90))
-    (property "Footprint" "" (id 2) (at 195.58 107.188 90)
+    (property "Footprint" "Resistor_SMD:R_0805_2012Metric_Pad1.20x1.40mm_HandSolder" (id 2) (at 195.58 107.188 90)
       (effects (font (size 1.27 1.27)) hide)
     )
@@
     (property "Reference" "J4" (id 0) (at 311.15 43.18 90))
     (property "Value" "Port D" (id 1) (at 311.15 45.72 90))
-    (property "Footprint" "" (id 2) (at 311.15 48.26 0)
+    (property "Footprint" "Connector_PinSocket_2.54mm:PinSocket_1x05_P2.54mm_Vertical" (id 2) (at 311.15 48.26 0)
       (effects (font (size 1.27 1.27)) hide)
     )
@@
       (effects (font (size 1.27 1.27)) (justify left))
     )
-    (property "Footprint" "" (id 2) (at 73.66 26.67 0)
-      (effects (font (size 1.27 1.27)) hide)
-    )
+    (property "Footprint" "Capacitor_SMD:C_0805_2012Metric" (id 2) (at 73.66 26.67 0)
+      (effects (font (size 1.27 1.27)) hide)
+    )

Commit message: Update custom_board.kicad_sch
Parts:
- removed SW2: Reset Button, symbol Switch:SW_Push
- added C?: .1u, symbol Device:C_Small
- added SW2: SW_Push_Dual, symbol Switch:SW_Push_Dual
- Y1: value (none) -> HighOscillator; footprint (none) -> Crystal:Crystal_SMD_Abracon_ABM10-4Pin_2.5x2.0mm
Connections:
- net GND: now also C?.2, SW2.2, SW2.4
- net at IC1.58 (~{RESET}), R3.1: now also C?.1, SW2.1, SW2.3
Changed lines of the file:
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@@
   (junction (at 207.01 107.95) (diameter 0) (color 0 0 0 0)
   )
+  (junction (at 217.17 134.62) (diameter 0) (color 0 0 0 0)
+  )
   (junction (at 199.39 105.41) (diameter 0) (color 0 0 0 0)
   )
@@
   (junction (at 205.74 86.36) (diameter 0) (color 0 0 0 0)
   )
+  (junction (at 198.12 134.62) (diameter 0) (color 0 0 0 0)
+  )
   (junction (at 25.4 24.13) (diameter 0) (color 0 0 0 0)
   )
@@
   )
   (junction (at 200.66 81.28) (diameter 0) (color 0 0 0 0)
+  )
+  (junction (at 207.01 134.62) (diameter 0) (color 0 0 0 0)
   )
   (junction (at 35.56 29.21) (diameter 0) (color 0 0 0 0)
@@
     (stroke (width 0) (type default) (color 0 0 0 0))
   )
+  (wire (pts (xy 217.17 129.54) (xy 217.17 134.62))
+    (stroke (width 0) (type default) (color 0 0 0 0))
+  )
   (wire (pts (xy 53.34 67.31) (xy 53.34 68.58))
     (stroke (width 0) (type default) (color 0 0 0 0))
@@
   )
   (wire (pts (xy 49.53 67.31) (xy 53.34 67.31))
+    (stroke (width 0) (type default) (color 0 0 0 0))
+  )
+  (wire (pts (xy 207.01 129.54) (xy 207.01 134.62))
     (stroke (width 0) (type default) (color 0 0 0 0))
   )
@@
     (pin "1")
   )
-  (symbol (lib_id "Switch:SW_Push") (at 212.09 134.62 0) (unit 1)
-    (in_bom yes) (on_board yes) (fields_autoplaced)
-    (property "Reference" "SW2" (id 0) (at 212.09 127 0))
-    (property "Value" "Reset Button" (id 1) (at 212.09 129.54 0))
-    (property "Footprint" "" (id 2) (at 212.09 129.54 0)
-      (effects (font (size 1.27 1.27)) hide)
-    )
-    (property "Datasheet" "~" (id 3) (at 212.09 129.54 0)
-      (effects (font (size 1.27 1.27)) hide)
-    )
-    (pin "1")
-    (pin "2")
-  )
   (symbol (lib_id "Device:C_Small") (at 205.74 105.41 90) (unit 1)
     (in_bom yes) (on_board yes) (fields_autoplaced)
@@
     (pin "1")
   )
+  (symbol (lib_id "power:GND") (at 198.12 139.7 0) (unit 1)
+    (in_bom yes) (on_board yes) (fields_autoplaced)
+    (property "Reference" "#PWR?" (id 0) (at 198.12 146.05 0)
+      (effects (font (size 1.27 1.27)) hide)
+    )
+    (property "Value" "GND" (id 1) (at 198.12 144.78 0))
+    (property "Footprint" "" (id 2) (at 198.12 139.7 0)
+      (effects (font (size 1.27 1.27)) hide)
+    )
+    (property "Datasheet" "" (id 3) (at 198.12 139.7 0)
+      (effects (font (size 1.27 1.27)) hide)
+    )
+    (pin "1")
+  )
+  (symbol (lib_id "Switch:SW_Push_Dual") (at 212.09 129.54 0) (unit 1)
+    (in_bom yes) (on_board yes) (fields_autoplaced)
+    (property "Reference" "SW2" (id 0) (at 212.09 121.92 0))
+    (property "Value" "SW_Push_Dual" (id 1) (at 212.09 124.46 0))
+    (property "Footprint" "" (id 2) (at 212.09 124.46 0)
+      (effects (font (size 1.27 1.27)) hide)
+    )
+    (property "Datasheet" "~" (id 3) (at 212.09 124.46 0)
+      (effects (font (size 1.27 1.27)) hide)
+    )
+    (pin "1")
+    (pin "2")
+    (pin "3")
+    (pin "4")
+  )
   (symbol (lib_id "power:GND") (at 142.24 157.48 0) (unit 1)
     (in_bom yes) (on_board yes) (fields_autoplaced)
@@
     )
     (pin "1")
+  )
+  (symbol (lib_id "Device:C_Small") (at 198.12 137.16 0) (unit 1)
+    (in_bom yes) (on_board yes)
+    (property "Reference" "C?" (id 0) (at 193.04 135.89 0)
+      (effects (font (size 1.27 1.27)) (justify left))
+    )
+    (property "Value" ".1u" (id 1) (at 193.04 138.43 0)
+      (effects (font (size 1.27 1.27)) (justify left))
+    )
+    (property "Footprint" "" (id 2) (at 198.12 137.16 0)
+      (effects (font (size 1.27 1.27)) hide)
+    )
+    (property "Datasheet" "~" (id 3) (at 198.12 137.16 0)
+      (effects (font (size 1.27 1.27)) hide)
+    )
+    (pin "1")
+    (pin "2")
   )
   (symbol (lib_id "power:+3V3") (at 92.71 92.71 90) (unit 1)
@@
     (in_bom yes) (on_board yes)
     (property "Reference" "Y1" (id 0) (at 201.93 104.14 90))
-    (property "Value" "" (id 1) (at 217.17 107.95 90))
-    (property "Footprint" "" (id 2) (at 199.39 107.95 0)
+    (property "Value" "HighOscillator" (id 1) (at 217.17 107.95 90))
+    (property "Footprint" "Crystal:Crystal_SMD_Abracon_ABM10-4Pin_2.5x2.0mm" (id 2) (at 199.39 107.95 0)
       (effects (font (size 1.27 1.27)) hide)
     )
@@
       (reference "#PWR0109") (unit 1) (value "+3V3") (footprint "")
     )
+    (path "/93fa6089-335f-4f46-88d4-ef4197169f92"
+      (reference "#PWR?") (unit 1) (value "GND") (footprint "")
+    )
     (path "/c1f0a81d-bdc1-4587-88e9-a039e356b3a4"
       (reference "C1") (unit 1) (value "1u") (footprint "Capacitor_SMD:C_0805_2012Metric")
@@
       (reference "C14") (unit 1) (value "10p") (footprint "Capacitor_SMD:C_0805_2012Metric")
     )
+    (path "/b75c0a99-dfe9-4bef-beb4-f39cedbd4d4f"
+      (reference "C?") (unit 1) (value ".1u") (footprint "")
+    )
     (path "/111eee09-5402-4318-928f-1b56881e0b97"
       (reference "IC1") (unit 1) (value "TMPM46BF10FG") (footprint "Package_DFN_QFN:TMPM_Custom_Footprint")
@@
       (reference "SW1") (unit 1) (value "Boot Switch") (footprint "")
     )
-    (path "/2c730731-dcf4-4552-9401-d14d23c54ec9"
-      (reference "SW2") (unit 1) (value "Reset Button") (footprint "")
+    (path "/9abf177a-1aaa-434f-b2c3-365691ca3d47"
+      (reference "SW2") (unit 1) (value "SW_Push_Dual") (footprint "")
     )
     (path "/eac2d247-2412-4b3d-b454-cddab0c7248a"

Commit message: idk
Parts:
- removed SW2: SW_Push_Dual, symbol Switch:SW_Push_Dual
- added SW2: SW_Push, Button_Switch_THT:Push_E-Switch_KS01Q01, symbol Switch:SW_Push
- C15: renamed from C?; footprint (none) -> Capacitor_SMD:C_0805_2012Metric
- SW1: footprint (none) -> Button_Switch_SMD:SW_DIP_SPSTx01_Slide_9.78x4.72mm_W8.61mm_P2.54mm
Connections:
- net GND: now also SW2.2
- net at C15.1, IC1.58 (~{RESET}), R3.1: now also SW2.1
Other:
- moved on the sheet: C13, C14, C15, C4, C5, IC1, J10, J11, J12, J2, J3, J4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
